File: Hardware/SparkFun_Qwiic_Navigation.kicad_pcb (KiCad board)
At the start: 2 copper layers, 25.4 x 25.4 mm, 68 parts, among them J1 Qwiic_RA, J2 Conn_01x04, J3 Qwiic_RA, J5 I2C, SW2 Nav Switch, U4 PCA9554PW

Commit message: Update SCH to v11
Parts:
- removed kibuzzard-66EF7B78: G***, kibuzzard-66EF7B78
- added kibuzzard-675B45F7: G***, kibuzzard-675B45F7, B.Cu at (152.7, 104.8)
- turned SW2 to 0 degrees
Routing:
- net SW_Center: track 6.29 -> 15.0 mm
- net SW_Right: track 18.1 -> 10.6 mm
- net SW_Down: track 14.7 -> 7.75 mm
- net SW_Left: track 14.3 -> 9.25 mm, vias 3 -> 1
- net SW_Up: track 10.2 -> 11.6 mm, vias 2 -> 1
Other:
- board text added: "v11"
- board text removed: "v10"
